Commit message: Enable guarded quadruped self-collision

File: robot-cad/exports/urdf/quadruped_robot.urdf (robot description, URDF)
Before this commit: robot st3215_quadruped, 13 links, 12 joints
Links:
- link front_left_distal_link: geometry collision box size=0.045223408 0.0378 0.024723408; collision box size=0.155285 0.035229 0.0713
- link front_left_hip_link: geometry collision box size=0.045223408 0.0378 0.024723408; collision box size=0.0713 0.127308 0.04805
- link front_left_proximal_link: geometry collision box size=0.045223408 0.0378 0.024723408; collision box size=0.155285 0.035229 0.0713
- link front_right_distal_link: geometry collision box size=0.045223408 0.0378 0.024723408; collision box size=0.155285 0.035229 0.0713
- link front_right_hip_link: geometry collision box size=0.045223408 0.0378 0.024723408; collision box size=0.0713 0.127308 0.04805
- link front_right_proximal_link: geometry collision box size=0.045223408 0.0378 0.024723408; collision box size=0.155285 0.035229 0.0713
- link rear_left_distal_link: geometry collision box size=0.045223408 0.0378 0.024723408; collision box size=0.155285 0.035229 0.0713
- link rear_left_hip_link: geometry collision box size=0.045223408 0.0378 0.024723408; collision box size=0.0713 0.127308 0.04805
- link rear_left_proximal_link: geometry collision box size=0.045223408 0.0378 0.024723408; collision box size=0.155285 0.035229 0.0713
- link rear_right_distal_link: geometry collision box size=0.045223408 0.0378 0.024723408; collision box size=0.155285 0.035229 0.0713
- link rear_right_hip_link: geometry collision box size=0.045223408 0.0378 0.024723408; collision box size=0.0713 0.127308 0.04805
- link rear_right_proximal_link: geometry collision box size=0.045223408 0.0378 0.024723408; collision box size=0.155285 0.035229 0.0713

Commit message: Connect mounted camera to Isaac Sim

File: robot-cad/exports/urdf/quadruped_robot.urdf (robot description, URDF)
Before this commit: robot st3215_quadruped, 13 links, 12 joints
Links:
- added link camera_link, mass 0.074635989; collision box size=0.016661073 0.048 0.045184589; collision box size=0.0215 0.038 0.038
- added link camera_optical_frame
Joints:
- added joint base_to_camera_mount: type fixed, parent base_link, child camera_link, origin xyz=0.09 0 0.1 rpy=0 0 0
- added joint camera_to_optical: type fixed, parent camera_link, child camera_optical_frame, origin xyz=0.0245 0 0.023 rpy=-1.570796327 0 -1.570796327

Commit message: Add body IMU mount and Isaac sensor

File: robot-cad/exports/urdf/quadruped_robot.urdf (robot description, URDF)
Before this commit: robot st3215_quadruped, 15 links, 14 joints
Links:
- added link imu_link, mass 0.0025; collision box size=0.0254 0.02286 0.00453; visual mesh filename=../stl/adafruit_bno085_stemma_qt.stl scale=0.001 0.001 0.001
Joints:
- added joint base_to_imu: type fixed, parent base_link, child imu_link, origin xyz=0 0 0.06516 rpy=0 0 0
